File: kicad/sr89_udk_registers.kicad_sch (KiCad schematic)
At the start: 0 parts

Commit message: routed, but not rules checked
Parts:
- added C127, C128, C129, C130, C131: 100n, Capacitor_SMD:C_0402_1005Metric, symbol ts-kicad-lib:C
- added C142, C143, C144, C145: 470µ, Capacitor_SMD:C_0603_1608Metric, symbol ts-kicad-lib:C
- added J1, J2: Conn_01x10_MountingPin, ts-flat-flex-cable:CONN_FH12-12S-0.5SH55_HIR, symbol Connector_Generic_MountingPin:Conn_01x12_MountingPin
- added J10, J14: QWIIC, Connector_JST:JST_SH_SM04B-SRSS-TB_1x04-1MP_P1.00mm_Horizontal, symbol ts-kicad-lib:QWIIC
- added J11, J17: ARGB, Connector_JST:JST_SH_SM03B-SRSS-TB_1x03-1MP_P1.00mm_Horizontal, symbol ts-kicad-lib:CONN_03
- added J12, J13: 5V, Connector_JST:JST_SH_SM02B-SRSS-TB_1x02-1MP_P1.00mm_Horizontal, symbol ts-kicad-lib:CONN_02
- added J15, J8: SPI, Connector_JST:JST_SH_SM06B-SRSS-TB_1x06-1MP_P1.00mm_Horizontal, symbol ts-kicad-lib:CONN_06
- added J16, J9: CONN, Connector_JST:JST_SH_SM05B-SRSS-TB_1x05-1MP_P1.00mm_Horizontal, symbol ts-kicad-lib:CONN_05
- added NT1, NT2: NetTie_2, ts-kicad-lib:NetTie-2_SMD_Pad0.254mm, symbol ts-kicad-lib:NetTie_2
- added Q1, Q2: 2N7002, Package_TO_SOT_SMD:SOT-23, symbol Transistor_FET:2N7002
- added R1, R2, R3, R4, R6, R7: 10K, Resistor_SMD:R_Array_Convex_4x0402, symbol ts-kicad-lib:R_Array04
- added R10, R5, R8, R9: 5K1, Resistor_SMD:R_0402_1005Metric, symbol ts-kicad-lib:R
- added U1, U2: 74HC595PW,118, Package_SO:TSSOP-16_4.4x5mm_P0.65mm, symbol ts-kicad-lib:74HC595
- added U3, U4, U5: MC74HC589, Package_SO:TSSOP-16_4.4x5mm_P0.65mm, symbol ts-kicad-lib:MC74HC589
Connections:
- new net: R7.5, U5.7 (H)
- new net: R10.1, U2.10 (~{SRCLR/MR})
- new net: R9.1, U1.10 (~{SRCLR/MR})
- new net: R7.7, U5.5 (F)
- new net: R6.8, U5.15 (A)
- new net: R7.6, U5.6 (G)
- new net 3V3^{1}: C127.1, C128.1, C129.1, J1.1 (Pin_1), J10.2, J8.2, R5.2, R9.2, U1.16 (Vcc), U3.16 (VCC), U4.16 (VCC)
- new net 3V3_{2}: C130.1, C131.1, J14.2, J15.2, J2.12 (Pin_12), R10.2, R8.2, U2.16 (Vcc), U5.16 (VCC)
- new net 5V^{1}: C142.1, C143.1, J1.11 (Pin_11), J1.12 (Pin_12), J11.3, J12.2
- new net 5V_{2}: C144.1, C145.1, J13.2, J17.3, J2.1 (Pin_1), J2.2 (Pin_2)
- new net COL0: R1.8, U3.15 (A)
- new net COL1: R1.7, U3.1 (B)
- new net COL10: R3.6, U4.2 (C)
- new net COL11: R3.5, U4.3 (D)
- new net COL12: R4.8, U4.4 (E)
- new net COL13: R4.7, U4.5 (F)
- new net COL14: R4.6, U4.6 (G)
- new net COL15: R4.5, U4.7 (H)
- new net COL2: R1.6, U3.2 (C)
- new net COL3: R1.5, U3.3 (D)
- new net COL4: R2.8, U3.4 (E)
- new net COL5: R2.7, U3.5 (F)
- new net COL6: R2.6, U3.6 (G)
- new net COL7: R2.5, U3.7 (H)
- new net COL8: R3.8, U4.15 (A)
- new net COL9: R3.7, U4.1 (B)
- new net COL_1_2: U3.14 (SA), U4.9 (QH)
- new net COL_2_3^{1}: J1.8 (Pin_8), U4.14 (SA)
- new net COL_2_3_{2}: J2.5 (Pin_5), NT2.2
- new net COL_CS^{1}: J1.5 (Pin_5), J9.1, Q1.1 (G), U3.10 (OE/~{CS}), U4.10 (OE/~{CS})
- new net COL_CS_{2}: J16.1, J2.8 (Pin_8), Q2.1 (G), U5.10 (OE/~{CS})
- new net COL_{2}0: R6.7, U5.1 (B)
- new net COL_{2}1: R6.6, U5.2 (C)
- new net COL_{2}2: R6.5, U5.3 (D)
- new net COL_{2}3: R7.8, U5.4 (E)
- new net GND^{1}: C127.2, C128.2, C129.2, C142.2, C143.2, J1.10 (Pin_10), J1.2 (Pin_2), J1.MP (MountPin), J10.1, J10.MP, J11.1, J11.MP, J12.1, J12.MP, J8.1, J8.MP, J9.MP, Q1.2 (S), R1.1, R1.2, R1.3, R1.4, R2.1, R2.2, R2.3, R2.4, R3.1, R3.2, R3.3, R3.4, R4.1, R4.2, R4.3, R4.4, U1.13 (~{OE}), U1.8 (GND), U3.8 (GND), U4.8 (GND)
- new net GND_{2}: C130.2, C131.2, C144.2, C145.2, J13.1, J13.MP, J14.1, J14.MP, J15.1, J15.MP, J16.MP, J17.1, J17.MP, J2.11 (Pin_11), J2.3 (Pin_3), J2.MP (MountPin), Q2.2 (S), R6.1, R6.2, R6.3, R6.4, R7.1, R7.2, R7.3, R7.4, U2.13 (~{OE}), U2.8 (GND), U5.14 (SA), U5.8 (GND)
- new net LATCH^{1}: Q1.3 (D), R5.1, U3.12 (LATCH), U3.13 (SS/~{PL}), U4.12 (LATCH), U4.13 (SS/~{PL})
- new net LATCH_{2}: Q2.3 (D), R8.1, U5.12 (LATCH), U5.13 (SS/~{PL})
- new net MISO^{1}: J8.4, U3.9 (QH)
- new net MISO_{2}: J15.4, NT2.1, U5.9 (QH)
- new net MOSI^{1}: J8.5, U1.14 (SER)
- new net MOSI_{2}: J15.5, NT1.1, U2.14 (SER)
- new net RGB^{1}: J11.2
- new net RGB_{2}: J17.2, J2.4 (Pin_4)
- new net ROW^{1}0: U1.1
- new net ROW^{1}1: U1.2
- new net ROW^{1}2: U1.3
- new net ROW^{1}3: U1.4
- new net ROW^{1}4: U1.5
- new net ROW^{1}5: U1.6
- new net ROW_1_2^{1}: J1.7 (Pin_7), U1.9 (QH'/7S)
- new net ROW_1_2_{2}: J2.6 (Pin_6), NT1.2
- new net ROW_CS^{1}: J1.4 (Pin_4), J9.2, U1.12 (RCLK/STCP)
- new net ROW_CS_{2}: J16.2, J2.9 (Pin_9), U2.12 (RCLK/STCP)
- new net ROW_{2}0: U2.1
- new net ROW_{2}1: U2.2
- new net ROW_{2}2: U2.3
- new net ROW_{2}3: U2.4
- new net ROW_{2}4: U2.5
- new net ROW_{2}5: U2.6
- new net SCK^{1}: J1.6 (Pin_6), J8.3, U1.11 (SRCLK/SHCP), U3.11 (SC/SCK), U4.11 (SC/SCK)
- new net SCK_{2}: J15.3, J2.7 (Pin_7), U2.11 (SRCLK/SHCP), U5.11 (SC/SCK)
- new net SCL^{1}: J10.4
- new net SCL_{2}: J14.4
- new net SDA^{1}: J10.3
- new net SDA_{2}: J14.3
- new net W127_{in}: J1.9 (Pin_9)
- new net ~{FAULT^{1}}: J9.5
- new net ~{FAULT_{2}}: J16.5
- new net ~{LED_EN^{1}}: J1.3 (Pin_3), J8.6
- new net ~{LED_EN_{2}}: J15.6, J2.10 (Pin_10)
- no-connect marks 0 -> 9
Other:
- note added: "SR110 Full-size Keyboard"
- note added: "SR21 Numpad Keyboard"
- note added: "SR89 TKL Keyboard"
